File: esp32wroomOled_V01/esp32wroomOled_V01.sch (KiCad schematic (older format))
At the start: 60 parts, among them IC1 MCP73811_2, J1 USB_B_Mini, J2 Conn_01x17, J3 Conn_01x17, J4 JST_2MM_MALE, Q1 DMG2307L, Q2 MMBT3904, Q3 MMBT3904, SW7 SW_Push_SPDT, SW8 RESET BTN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

Commit message: Add files via upload
Changed lines of the file:
@@
 Text Notes 900  750  0    118  Italic 0
 ESP-32S-WROOM
-Text Label 950  1650 1    60   ~ 0
-ESP_RST
 $Comp
 L LED_ALT LED1
@@
 Text Label 4800 3450 2    60   ~ 0
 ESP_RST
-Text Label 950  1950 3    60   ~ 0
-MPU_INT
 $Comp
 L SW_Push_SPDT SW7
@@
 	7400 5600 7450 5600
 Wire Wire Line
-	6950 5600 7100 5600
-Wire Wire Line
-	6950 6150 7100 6150
+	6950 5600 7000 5600
+Wire Wire Line
+	7000 5600 7100 5600
+Wire Wire Line
+	6950 6150 7050 6150
+Wire Wire Line
+	7050 6150 7100 6150
 Wire Wire Line
 	7750 5800 7750 5850
@@
 	7250 5350 7250 5300
 Wire Wire Line
-	7650 5350 7900 5350
+	7650 5350 7750 5350
+Wire Wire Line
+	7750 5350 7900 5350
 Wire Wire Line
 	7750 5350 7750 5400
@@
 	10300 3650 10450 3650
 Wire Wire Line
-	10300 750  10300 3900
+	10300 750  10300 1450
+Wire Wire Line
+	10300 1450 10300 1650
+Wire Wire Line
+	10300 1650 10300 1850
+Wire Wire Line
+	10300 1850 10300 1950
+Wire Wire Line
+	10300 1950 10300 2150
+Wire Wire Line
+	10300 2150 10300 2250
+Wire Wire Line
+	10300 2250 10300 2350
+Wire Wire Line
+	10300 2350 10300 2750
+Wire Wire Line
+	10300 2750 10300 2850
+Wire Wire Line
+	10300 2850 10300 2950
+Wire Wire Line
+	10300 2950 10300 3050
+Wire Wire Line
+	10300 3050 10300 3150
+Wire Wire Line
+	10300 3150 10300 3550
+Wire Wire Line
+	10300 3550 10300 3650
+Wire Wire Line
+	10300 3650 10300 3850
+Wire Wire Line
+	10300 3850 10300 3900
 Wire Wire Line
 	10450 3550 10300 3550
@@
 	10450 1250 9700 1250
 Wire Wire Line
-	9700 750  9700 1750
-Wire Wire Line
-	8950 1550 10450 1550
+	9700 750  9700 1250
+Wire Wire Line
+	9700 1250 9700 1550
+Wire Wire Line
+	9700 1550 9700 1750
+Wire Wire Line
+	8950 1550 9250 1550
+Wire Wire Line
+	9250 1550 9550 1550
+Wire Wire Line
+	9550 1550 9700 1550
+Wire Wire Line
+	9700 1550 10450 1550
 Connection ~ 9700 1250
 Wire Wire Line
@@
 Connection ~ 9700 1550
 Wire Wire Line
-	10050 3150 10050 3550
+	10050 3150 10050 3450
+Wire Wire Line
+	10050 3450 10050 3550
 Wire Wire Line
 	10050 3850 10050 3750
 Wire Wire Line
-	8950 3850 10300 3850
+	8950 3850 9150 3850
+Wire Wire Line
+	9150 3850 9400 3850
+Wire Wire Line
+	9400 3850 9600 3850
+Wire Wire Line
+	9600 3850 9800 3850
+Wire Wire Line
+	9800 3850 10050 3850
+Wire Wire Line
+	10050 3850 10300 3850
 Connection ~ 10300 3850
 Wire Wire Line
@@
 	9600 3350 10450 3350
 Wire Wire Line
-	9800 3450 10450 3450
+	9800 3450 10050 3450
+Wire Wire Line
+	10050 3450 10450 3450
 Wire Wire Line
 	9400 3800 9400 3850
@@
 Connection ~ 9400 3850
 Wire Wire Line
-	9150 2050 10450 2050
+	9150 2050 9250 2050
+Wire Wire Line
+	9250 2050 9550 2050
+Wire Wire Line
+	9550 2050 10450 2050
 Wire Wire Line
 	9150 2050 9150 3550
@@
 	10450 2450 9950 2450
 Wire Wire Line
-	9950 2550 10450 2550
+	9950 2550 10150 2550
+Wire Wire Line
+	10150 2550 10450 2550
 Wire Wire Line
 	10450 2650 10150 2650
@@
 	11000 4700 10900 4700
 Wire Wire Line
-	11000 4300 11000 5950
+	11000 4300 11000 4500
+Wire Wire Line
+	11000 4500 11000 4700
+Wire Wire Line
+	11000 4700 11000 4900
+Wire Wire Line
+	11000 4900 11000 5100
+Wire Wire Line
+	11000 5100 11000 5300
+Wire Wire Line
+	11000 5300 11000 5950
 Wire Wire Line
 	10900 4900 11000 4900
@@
 Connection ~ 11000 5100
 Wire Wire Line
-	8400 4700 10600 4700
-Wire Wire Line
-	8400 4900 10600 4900
+	8400 4700 9100 4700
+Wire Wire Line
+	9100 4700 10600 4700
+Wire Wire Line
+	8400 4900 9350 4900
+Wire Wire Line
+	9350 4900 10600 4900
 Wire Wire Line
 	9100 6200 9100 6250
 Wire Wire Line
-	8600 6250 11000 6250
-Wire Wire Line
-	11000 6150 11000 6300
+	8600 6250 8850 6250
+Wire Wire Line
+	8850 6250 9350 6250
+Wire Wire Line
+	9350 6250 9600 6250
+Wire Wire Line
+	9600 6250 9850 6250
+Wire Wire Line
+	9850 6250 11000 6250
+Wire Wire Line
+	11000 6150 11000 6250
+Wire Wire Line
+	11000 6250 11000 6300
 Wire Wire Line
 	9350 6250 9350 6200
@@
 	7650 4700 7500 4700
 Wire Wire Line
-	7650 4350 7650 4700
+	7650 4350 7650 4500
+Wire Wire Line
+	7650 4500 7650 4700
 Wire Wire Line
 	7500 4500 7650 4500
@@
 	3300 1500 3200 1500
 Wire Wire Line
-	3300 1050 3300 1500
+	3300 1050 3300 1400
+Wire Wire Line
+	3300 1400 3300 1500
 Wire Wire Line
 	3300 1050 3450 1050
 Wire Wire Line
-	3450 800  3450 1150
+	3450 800  3450 1050
+Wire Wire Line
+	3450 1050 3450 1150
 Wire Wire Line
 	3200 1400 3300 1400
@@
 Connection ~ 11000 4700
 Wire Wire Line
-	8400 4500 10600 4500
+	8400 4500 8850 4500
+Wire Wire Line
+	8850 4500 10600 4500
 Wire Wire Line
 	10900 5300 11000 5300
@@
 Connection ~ 11000 4500
 Wire Wire Line
-	8400 4300 10600 4300
+	8400 4300 8600 4300
+Wire Wire Line
+	8600 4300 10600 4300
 Wire Wire Line
 	8600 6200 8600 6250
@@
 Connection ~ 8850 4500
 Wire Wire Line
-	2650 7250 2650 7450
+	2650 7250 2650 7350
+Wire Wire Line
+	2650 7350 2650 7450
 Wire Wire Line
 	2500 7250 2650 7250
@@
 	1100 5850 800  5850
 Wire Wire Line
-	800  5750 800  6150
+	800  5750 800  5850
+Wire Wire Line
+	800  5850 800  6150
 Wire Wire Line
 	1100 5750 800  5750
@@
 Connection ~ 3100 6650
 Wire Wire Line
-	3100 5800 3100 6700
+	3100 5800 3100 5850
+Wire Wire Line
+	3100 5850 3100 6050
+Wire Wire Line
+	3100 6050 3100 6650
+Wire Wire Line
+	3100 6650 3100 6700
 Wire Wire Line
 	3000 5850 3100 5850
@@
 	2700 6650 3100 6650
 Wire Wire Line
-	5950 5550 6350 5550
-Wire Wire Line
-	6350 5500 6350 5650
+	5950 5550 6150 5550
+Wire Wire Line
+	6150 5550 6350 5550
+Wire Wire Line
+	6350 5500 6350 5550
+Wire Wire Line
+	6350 5550 6350 5650
 Wire Wire Line
 	6150 5650 6150 5550
@@
 	5150 5750 5100 5750
 Wire Wire Line
-	5100 5750 5100 5900
-Wire Wire Line
-	3900 5450 3900 5600
+	5100 5750 5100 5850
+Wire Wire Line
+	5100 5850 5100 5900
+Wire Wire Line
+	3900 5450 3900 5550
+Wire Wire Line
+	3900 5550 3900 5600
 Wire Wire Line
 	4100 5550 4100 5750
@@
 Connection ~ 3900 5550
 Wire Wire Line
-	3450 5150 3450 5600
+	3450 5150 3450 5250
+Wire Wire Line
+	3450 5250 3450 5550
+Wire Wire Line
+	3450 5550 3450 5600
 Wire Wire Line
 	3450 5550 3500 5550
@@
 	4050 7350 4500 7350
 Wire Wire Line
-	4000 6300 4000 6800
+	4000 6300 4000 6450
+Wire Wire Line
+	4000 6450 4000 6800
 Wire Wire Line
 	4000 6800 4100 6800
@@
 	5200 6800 5600 6800
 Wire Wire Line
-	5600 6700 5600 7150
+	5600 6700 5600 6800
+Wire Wire Line
+	5600 6800 5600 7150
 Connection ~ 5600 6800
 Wire Notes Line
@@
 	1000 1850 1350 1850
 Wire Wire Line
-	950  1950 1350 1950
+	1000 1950 1350 1950
 Wire Wire Line
 	1000 2150 1350 2150
@@
 	850  3800 850  550
 Wire Wire Line
-	1900 6850 2600 6850
+	1900 6850 2500 6850
+Wire Wire Line
+	2500 6850 2600 6850
 Connection ~ 2500 6850
 Wire Wire Line
@@
 	5200 7000 5300 7000
 Wire Wire Line
-	5300 7000 5300 7450
+	5300 7000 5300 7350
+Wire Wire Line
+	5300 7350 5300 7450
 Wire Wire Line
 	4100 7200 4050 7200
@@
 	6050 6650 6050 6700
 Wire Wire Line
-	6050 7000 6050 7100
+	6050 7000 6050 7050
+Wire Wire Line
+	6050 7050 6050 7100
 Wire Wire Line
 	6050 7400 6050 7450
@@
 	4350 3550 4450 3550
 Wire Wire Line
-	4750 3550 4850 3550
+	4750 3550 4800 3550
+Wire Wire Line
+	4800 3550 4850 3550
 Wire Wire Line
 	5150 3550 5200 3550
@@
 	4800 3850 4800 3800
 Wire Wire Line
-	4800 3450 4800 3600
+	4800 3450 4800 3550
+Wire Wire Line
+	4800 3550 4800 3600
 Connection ~ 4800 3550
 Wire Notes Line
@@
 	4200 4100 5350 4100
 Wire Wire Line
-	3800 5550 5150 5550
+	3800 5550 3900 5550
+Wire Wire Line
+	3900 5550 4100 5550
+Wire Wire Line
+	4100 5550 5150 5550
 Wire Wire Line
 	2100 4950 1750 4950
@@
 	2550 3200 2550 3550
 Wire Wire Line
-	8400 5100 10550 5100
-Wire Wire Line
-	8400 5300 10600 5300
+	8400 5100 9600 5100
+Wire Wire Line
+	9600 5100 10550 5100
+Wire Wire Line
+	8400 5300 9850 5300
+Wire Wire Line
+	9850 5300 10600 5300
 Wire Wire Line
 	9600 6200 9600 6250
@@
 Connection ~ 5100 5850
 Wire Wire Line
-	4550 5650 5150 5650
+	4550 5650 4650 5650
+Wire Wire Line
+	4650 5650 5150 5650
 Wire Wire Line
 	4100 5750 4150 5750
@@
 	4650 5850 4650 5650
 Connection ~ 4650 5650
+Text Label 950  1650 1    60   ~ 0
+ESP_RST
 $EndSCHEMATC
